Commit message: cleanup

File: src/SLAM/summit/summit_xl_common/summit_xl_description/robots/summit_xl_std.urdf.xacro (robot description, xacro)
@@ -71,5 +71,5 @@
 		<!-- ptz camera -->
 		<xacro:sensor_axis prefix="$(arg prefix)front_ptz_camera" parent="$(arg prefix)base_link">
-			<origin xyz="0.19 0 0.26" rpy="0 ${15*PI/180} 0"/>
+			<origin xyz="0.0 0.0 0.3" rpy="0 0 0"/>
 		</xacro:sensor_axis>
 	  <!-- RGBD -->
